File: LX200V20_test.sch (EAGLE design)
At the start: 3 parts

Commit message: First rough layout.
Parts:
- added C1, C2: 0.1uF, resistor:C-EUC0402
- added C3: EFI Capacitor (1000 pF, 2kV), resistor:C-EUC1206
- added C4: 330pF 50V, resistor:C-EUC0805
- added C5, C6: 0.01uF 250V, resistor:C-EUC0805
- added JP1: (no value), SparkFun-Connectors:M083.5MM-8
- added LED1, LED2, LED3, LED4: (no value), led:LEDCHIPLED_0603
- added R1, R2, R3, R4: 75, resistor:R-US_R0603
- added R10, R9: 4.7K 1/4W, resistor:R-US_R1206
- added R5, R6, R8: 130, resistor:R-US_R0603
- added R7: 470, resistor:R-US_R0603
- added STANDOFF1, STANDOFF2, STANDOFF3: STAND-OFF, SparkFun-Electromechanical:STAND-OFF
- added U$4: PT61017PEL, BlueRobotics-Main:PT61017PEL
- added U$5: TVS-SP4021, BlueRobotics-Main:TVS-SP4021
- added U$6: TETHER-HEADERSERIAL, BlueRobotics-Main:TETHER-HEADERSERIAL
- added U$7, U$8: HEADER-2POWER, BlueRobotics-Main:HEADER-2POWER
Connections:
- new net +3.3V: R5.1, R6.1, R7.1, U$1.3.3VD
- new net AC_CPLD_L: R10.2, U$3.PL_N, U$5.P$1
- new net AC_CPLD_N: R9.2, U$3.PL_L, U$5.P$2
- new net ETH-RX+: U$2.3, U$4.RX+
- new net ETH-RX-: U$2.6, U$4.RX-
- new net ETH-TX+: U$2.1, U$4.TX+
- new net ETH-TX-: U$2.2, U$4.TX-
- new net EXT_AC_A: C5.2, JP1.3
- new net EXT_AC_B: C6.2, JP1.4
- new net GND: C1.2, C2.2, C3.2, LED3.C, LED4.C, U$1.GND
- new net LED-ACT: R8.1
- new net LED-LINK: LED1.C, U$1.GPIO0
- new net LED-SELFCHECK: LED2.C, U$1.GPIO1
- new net LED2: U$1.GPIO2
- new net N$1: R1.2, U$4.CT-RX
- new net N$10: U$1.GPIO3
- new net N$11: C6.1, R10.1
- new net N$12: C5.1, R9.1
- new net N$2: R2.2, U$4.CT-TX
- new net N$3: R4.2, U$2.7, U$2.8
- new net N$4: C3.1, R1.1, R2.1, R3.1, R4.1
- new net N$5: R3.2, U$2.4, U$2.5
- new net N$6: LED1.A, R5.2
- new net N$7: LED2.A, R6.2
- new net N$8: LED3.A, R7.2
- new net N$9: LED4.A, R8.2
- new net PE-RD+: U$1.PERX_P, U$4.RD+
- new net PE-RD-: U$1.PERX_N, U$4.RD-
- new net PE-TD+: U$1.PETX_P, U$4.TD+
- new net PE-TD-: U$1.PETX_N, U$4.TD-
- new net RX+: U$1.RX+, U$3.RX+
- new net RX-: U$1.RX-, U$3.RX-
- new net TX+: C4.1, U$1.TX+, U$3.TX+
- new net TX-: C4.2, U$1.TX-, U$3.TX-
- new net VDD2P0: C1.1, C2.1, U$1.VDD2P0, U$4.CT-RD, U$4.CT-TD
- new net ZC_IN_EX: U$1.ZC_IN_EX
Other:
- note added: "Capacitor per HL1102 datasheet."
- note added: "SP4021-01FTG-C"
- moved on the sheet: U$1, U$2, U$3

Commit message: Updated layout.
Parts:
- added STANDOFF5: STAND-OFF, SparkFun-Electromechanical:STAND-OFF
- added U$9: VREG-OKI-78SR, BlueRobotics-Main:VREG-OKI-78SR
Connections:
- removed net LED2: U$1.GPIO2
- net LED-ACT: now also U$1.GPIO2
Changed lines of the file:
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@@
 <part name="STANDOFF2" library="SparkFun-Electromechanical" deviceset="STAND-OFF" device=""/>
 <part name="STANDOFF3" library="SparkFun-Electromechanical" deviceset="STAND-OFF" device=""/>
+<part name="STANDOFF5" library="SparkFun-Electromechanical" deviceset="STAND-OFF" device=""/>
+<part name="U$9" library="BlueRobotics-Main" deviceset="VREG-OKI-78SR" device=""/>
 </parts>
 <sheets>
@@
 <instance part="STANDOFF2" gate="G$1" x="238.76" y="190.5"/>
 <instance part="STANDOFF3" gate="G$1" x="238.76" y="198.12"/>
+<instance part="STANDOFF5" gate="G$1" x="231.14" y="198.12"/>
+<instance part="U$9" gate="G$1" x="193.04" y="233.68"/>
 </instances>
 <busses>
@@
 </segment>
 </net>
-<net name="LED2" class="0">
+<net name="LED-ACT" class="0">
+<segment>
+<pinref part="R8" gate="G$1" pin="1"/>
+<wire x1="198.12" y1="132.08" x2="185.42" y2="132.08" width="0.1524" layer="91"/>
+<label x="185.42" y="132.08" size="1.778" layer="95"/>
+</segment>
 <segment>
 <pinref part="U$1" gate="G$1" pin="GPIO2"/>
@@
 </segment>
 </net>
-<net name="LED-ACT" class="0">
-<segment>
-<pinref part="R8" gate="G$1" pin="1"/>
-<wire x1="198.12" y1="132.08" x2="185.42" y2="132.08" width="0.1524" layer="91"/>
-<label x="185.42" y="132.08" size="1.778" layer="95"/>
-</segment>
-</net>

Commit message: Removed AC components for DC-only support.
Parts:
- removed C5: 0.01uF 250V, resistor:C-EUC0805
- removed R9: 4.7K 1/4W, resistor:R-US_R1206
- C6: value 0.01uF 250V -> 0.01uF 500V; device resistor:C-EUC0805 -> resistor:C-EUC1206
- R10: value 4.7K 1/4W -> 10 1/4W
Connections:
- removed net AC_CPLD_N: R9.2, U$3.PL_L, U$5.P$2
- removed net N$12: C5.1, R9.1
- net EXT_AC_A: no longer C5.2
- net GND: now also U$3.PL_L, U$5.P$2
Changed lines of the file:
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@@
 <grid distance="0.1" unitdist="inch" unit="inch" style="lines" multiple="1" display="no" altdistance="0.01" altunitdist="inch" altunit="inch"/>
 <layers>
-<layer number="1" name="Top" color="4" fill="1" visible="no" active="no"/>
-<layer number="2" name="Route2" color="1" fill="3" visible="no" active="no"/>
-<layer number="3" name="Route3" color="4" fill="3" visible="no" active="no"/>
-<layer number="14" name="Route14" color="1" fill="6" visible="no" active="no"/>
-<layer number="15" name="Route15" color="4" fill="6" visible="no" active="no"/>
-<layer number="16" name="Bottom" color="1" fill="1" visible="no" active="no"/>
-<layer number="17" name="Pads" color="2" fill="1" visible="no" active="no"/>
-<layer number="18" name="Vias" color="2" fill="1" visible="no" active="no"/>
-<layer number="19" name="Unrouted" color="6" fill="1" visible="no" active="no"/>
-<layer number="20" name="Dimension" color="15" fill="1" visible="no" active="no"/>
-<layer number="21" name="tPlace" color="7" fill="1" visible="no" active="no"/>
-<layer number="22" name="bPlace" color="7" fill="1" visible="no" active="no"/>
-<layer number="23" name="tOrigins" color="15" fill="1" visible="no" active="no"/>
-<layer number="24" name="bOrigins" color="15" fill="1" visible="no" active="no"/>
-<layer number="25" name="tNames" color="7" fill="1" visible="no" active="no"/>
-<layer number="26" name="bNames" color="7" fill="1" visible="no" active="no"/>
-<layer number="27" name="tValues" color="7" fill="1" visible="no" active="no"/>
-<layer number="28" name="bValues" color="7" fill="1" visible="no" active="no"/>
+<layer number="1" name="Top" color="4" fill="1" visible="yes" active="no"/>
+<layer number="2" name="Route2" color="1" fill="3" visible="yes" active="no"/>
+<layer number="3" name="Route3" color="4" fill="3" visible="yes" active="no"/>
+<layer number="14" name="Route14" color="1" fill="6" visible="yes" active="no"/>
+<layer number="15" name="Route15" color="4" fill="6" visible="yes" active="no"/>
+<layer number="16" name="Bottom" color="1" fill="1" visible="yes" active="no"/>
+<layer number="17" name="Pads" color="2" fill="1" visible="yes" active="no"/>
+<layer number="18" name="Vias" color="2" fill="1" visible="yes" active="no"/>
+<layer number="19" name="Unrouted" color="6" fill="1" visible="yes" active="no"/>
+<layer number="20" name="Dimension" color="15" fill="1" visible="yes" active="no"/>
+<layer number="21" name="tPlace" color="7" fill="1" visible="yes" active="no"/>
+<layer number="22" name="bPlace" color="7" fill="1" visible="yes" active="no"/>
+<layer number="23" name="tOrigins" color="15" fill="1" visible="yes" active="no"/>
+<layer number="24" name="bOrigins" color="15" fill="1" visible="yes" active="no"/>
+<layer number="25" name="tNames" color="7" fill="1" visible="yes" active="no"/>
+<layer number="26" name="bNames" color="7" fill="1" visible="yes" active="no"/>
+<layer number="27" name="tValues" color="7" fill="1" visible="yes" active="no"/>
+<layer number="28" name="bValues" color="7" fill="1" visible="yes" active="no"/>
 <layer number="29" name="tStop" color="7" fill="3" visible="no" active="no"/>
 <layer number="30" name="bStop" color="7" fill="6" visible="no" active="no"/>
@@
 <layer number="35" name="tGlue" color="7" fill="4" visible="no" active="no"/>
 <layer number="36" name="bGlue" color="7" fill="5" visible="no" active="no"/>
-<layer number="37" name="tTest" color="7" fill="1" visible="no" active="no"/>
-<layer number="38" name="bTest" color="7" fill="1" visible="no" active="no"/>
+<layer number="37" name="tTest" color="7" fill="1" visible="yes" active="no"/>
+<layer number="38" name="bTest" color="7" fill="1" visible="yes" active="no"/>
 <layer number="39" name="tKeepout" color="4" fill="11" visible="no" active="no"/>
 <layer number="40" name="bKeepout" color="1" fill="11" visible="no" active="no"/>
@@
 <layer number="44" name="Drills" color="7" fill="1" visible="no" active="no"/>
 <layer number="45" name="Holes" color="7" fill="1" visible="no" active="no"/>
-<layer number="46" name="Milling" color="3" fill="1" visible="no" active="no"/>
-<layer number="47" name="Measures" color="7" fill="1" visible="no" active="no"/>
-<layer number="48" name="Document" color="7" fill="1" visible="no" active="no"/>
-<layer number="49" name="Reference" color="7" fill="1" visible="no" active="no"/>
-<layer number="50" name="dxf" color="7" fill="1" visible="no" active="no"/>
-<layer number="51" name="tDocu" color="7" fill="1" visible="no" active="no"/>
-<layer number="52" name="bDocu" color="7" fill="1" visible="no" active="no"/>
-<layer number="53" name="tGND_GNDA" color="7" fill="9" visible="no" active="no"/>
-<layer number="54" name="bGND_GNDA" color="1" fill="9" visible="no" active="no"/>
-<layer number="56" name="wert" color="7" fill="1" visible="no" active="no"/>
-<layer number="57" name="tCAD" color="7" fill="1" visible="no" active="no"/>
+<layer number="46" name="Milling" color="3" fill="1" visible="yes" active="no"/>
+<layer number="47" name="Measures" color="7" fill="1" visible="yes" active="no"/>
+<layer number="48" name="Document" color="7" fill="1" visible="yes" active="no"/>
+<layer number="49" name="Reference" color="7" fill="1" visible="yes" active="no"/>
+<layer number="50" name="dxf" color="7" fill="1" visible="yes" active="no"/>
+<layer number="51" name="tDocu" color="7" fill="1" visible="yes" active="no"/>
+<layer number="52" name="bDocu" color="7" fill="1" visible="yes" active="no"/>
+<layer number="53" name="tGND_GNDA" color="7" fill="9" visible="yes" active="no"/>
+<layer number="54" name="bGND_GNDA" color="1" fill="9" visible="yes" active="no"/>
+<layer number="56" name="wert" color="7" fill="1" visible="yes" active="no"/>
+<layer number="57" name="tCAD" color="7" fill="1" visible="yes" active="no"/>
 <layer number="90" name="Modules" color="5" fill="1" visible="yes" active="yes"/>
 <layer number="91" name="Nets" color="2" fill="1" visible="yes" active="yes"/>
@@
 <part name="R8" library="resistor" deviceset="R-US_" device="R0603" value="130"/>
 <part name="GND6" library="supply1" deviceset="GND" device=""/>
-<part name="R9" library="resistor" deviceset="R-US_" device="R1206" value="4.7K 1/4W"/>
-<part name="R10" library="resistor" deviceset="R-US_" device="R1206" value="4.7K 1/4W"/>
-<part name="C5" library="resistor" deviceset="C-EU" device="C0805" value="0.01uF 250V"/>
-<part name="C6" library="resistor" deviceset="C-EU" device="C0805" value="0.01uF 250V"/>
+<part name="R10" library="resistor" deviceset="R-US_" device="R1206" value="10 1/4W"/>
+<part name="C6" library="resistor" deviceset="C-EU" device="C1206" value="0.01uF 500V"/>
 <part name="FRAME1" library="BlueRobotics-Main" deviceset="FRAME-BLUEROBOTICS" device=""/>
 <part name="U$5" library="BlueRobotics-Main" deviceset="TVS-SP4021" device=""/>
@@
 <part name="STANDOFF5" library="SparkFun-Electromechanical" deviceset="STAND-OFF" device=""/>
 <part name="U$9" library="BlueRobotics-Main" deviceset="VREG-OKI-78SR" device=""/>
+<part name="GND7" library="supply1" deviceset="GND" device=""/>
 </parts>
 <sheets>
@@
 <instance part="R8" gate="G$1" x="203.2" y="132.08"/>
 <instance part="GND6" gate="1" x="223.52" y="127"/>
-<instance part="R9" gate="G$1" x="205.74" y="68.58" rot="R180"/>
 <instance part="R10" gate="G$1" x="205.74" y="43.18" rot="R180"/>
-<instance part="C5" gate="G$1" x="220.98" y="68.58" rot="R90"/>
 <instance part="C6" gate="G$1" x="220.98" y="43.18" rot="R90"/>
 <instance part="FRAME1" gate="G$1" x="0" y="0"/>
@@
 <instance part="STANDOFF5" gate="G$1" x="231.14" y="198.12"/>
 <instance part="U$9" gate="G$1" x="193.04" y="233.68"/>
+<instance part="GND7" gate="1" x="203.2" y="63.5"/>
 </instances>
 <busses>
@@
 <wire x1="58.42" y1="220.98" x2="40.64" y2="220.98" width="0.1524" layer="91"/>
 <label x="40.64" y="220.98" size="1.778" layer="95"/>
+</segment>
+<segment>
+<pinref part="U$3" gate="G$1" pin="PL_L"/>
+<label x="142.24" y="68.58" size="1.778" layer="95"/>
+<wire x1="139.7" y1="68.58" x2="175.26" y2="68.58" width="0.1524" layer="91"/>
+<pinref part="U$5" gate="G$1" pin="P$2"/>
+<wire x1="175.26" y1="68.58" x2="203.2" y2="68.58" width="0.1524" layer="91"/>
+<wire x1="175.26" y1="63.5" x2="175.26" y2="68.58" width="0.1524" layer="91"/>
+<junction x="175.26" y="68.58"/>
+<pinref part="GND7" gate="1" pin="GND"/>
+<wire x1="203.2" y1="68.58" x2="203.2" y2="66.04" width="0.1524" layer="91"/>
 </segment>
 </net>
@@
 </segment>
 </net>
-<net name="AC_CPLD_N" class="0">
-<segment>
-<pinref part="U$3" gate="G$1" pin="PL_L"/>
-<label x="142.24" y="68.58" size="1.778" layer="95"/>
-<wire x1="139.7" y1="68.58" x2="175.26" y2="68.58" width="0.1524" layer="91"/>
-<pinref part="R9" gate="G$1" pin="2"/>
-<pinref part="U$5" gate="G$1" pin="P$2"/>
-<wire x1="175.26" y1="68.58" x2="200.66" y2="68.58" width="0.1524" layer="91"/>
-<wire x1="175.26" y1="63.5" x2="175.26" y2="68.58" width="0.1524" layer="91"/>
-<junction x="175.26" y="68.58"/>
-</segment>
-</net>
 <net name="N$6" class="0">
 <segment>
@@
 </segment>
 </net>
-<net name="N$12" class="0">
-<segment>
-<pinref part="R9" gate="G$1" pin="1"/>
-<pinref part="C5" gate="G$1" pin="1"/>
-<wire x1="210.82" y1="68.58" x2="218.44" y2="68.58" width="0.1524" layer="91"/>
-</segment>
-</net>
 <net name="EXT_AC_A" class="0">
 <segment>
-<pinref part="C5" gate="G$1" pin="2"/>
-<wire x1="226.06" y1="68.58" x2="243.84" y2="68.58" width="0.1524" layer="91"/>
-<label x="231.14" y="68.58" size="1.778" layer="95"/>
-</segment>
-<segment>
 <wire x1="58.42" y1="251.46" x2="40.64" y2="251.46" width="0.1524" layer="91"/>

Commit message: Changing to Ethernet+Power only design.
Parts:
- added C5: 10uF, resistor:C-USC1206
- R10: value 10 1/4W -> 10 1/4W HV
- U$2: device SparkFun-Connectors:RJ45-8PTH -> BlueRobotics-Main:RJ45-8PTH
- U$3: value PLC10005345 -> UT11403S; device BlueRobotics-Main:PLC10005345 -> BlueRobotics-Main:UT11403S
- U$9: value VREG-OKI-78SR -> OKI-78SR-3.3V
Connections:
- net AC_CPLD_L renamed PL_N
- net EXT_AC_B renamed HV_SIGNAL
- removed net EXT_AC_A: JP1.3
- new net 3.3V: C5.1, U$9.OUT
- new net GNDI: JP1.3, U$3.PL_L, U$5.P$2
- new net VIN: U$7.2, U$9.IN
- net GND: now also C5.2, U$7.1, U$9.GND; no longer U$3.PL_L, U$5.P$2
Other:
- note added: "Connector: NPPN201BFLC-RC"
