File: fathom-x.kicad_sch (KiCad schematic)
At the start: 23 parts, among them IC1 1117-3.3V

Commit message: Updated Fathom-X Eagle parts to Kicad
Parts:
- removed U$1: LX200V20, Fathom-X:LX200V20, symbol Fathom-X-eagle-import:LX200V20
- removed U$2: UT11403S, Fathom-X:UT11403S, symbol Fathom-X-eagle-import:UT11403S
- added T1: UT11403S, Fathom-X:UT11403S, symbol BR_Inductors:UT11403S
- added U1: LX200V20-SOCKET, Fathom-X:LX200V20, symbol BR_Modules:LX200V20-SOCKET
- LED1, LED2: footprint Fathom-X:CHIPLED_0603 -> BR_Optoelectronics:LED_0603_1608Metric; symbol Fathom-X-eagle-import:LEDCHIPLED_0603 -> BR_Optoelectronic:LTST-C191KGKT; Manufacturer (none) -> Lite-On Inc.; Manufacturer Part Num (none) -> LTST-C191KGKT; Supplier 1 (none) -> DigiKey; Supplier 2 (none) -> DigiKey; Supplier 3 (none) -> JLCPCB; Supplier Part Num 1 (none) -> 160-1446-1-ND; Supplier Part Num 2 (none) -> 160-1446-2-ND; Supplier Part Num 3 (none) -> C125098
- R1: footprint Fathom-X:R0603 -> BR_Passives:R_0402_1005Metric; symbol Fathom-X-eagle-import:R-US_R0603 -> BR_Resistors_0402:R_0402_130R; Manufacturer (none) -> YAGEO; Manufacturer Part Num (none) -> RC0402FR-07130RL; Supplier 1 (none) -> DigiKey; Supplier 2 (none) -> Mouser; Supplier 3 (none) -> JLCPCB; Supplier Part Num 1 (none) -> 311-130LRCT-ND; Supplier Part Num 2 (none) -> 603-RC0402FR-07130RL; Supplier Part Num 3 (none) -> C477610
- R2: footprint Fathom-X:R0603 -> BR_Passives:R_0402_1005Metric; symbol Fathom-X-eagle-import:R-US_R0603 -> BR_Resistors_0402:R_0402_470R; Manufacturer (none) -> YAGEO; Manufacturer Part Num (none) -> RC0402FR-07470RL; Supplier 1 (none) -> DigiKey; Supplier 2 (none) -> DigiKey; Supplier 3 (none) -> JLCPCB; Supplier Part Num 1 (none) -> 311-470LRCT-ND; Supplier Part Num 2 (none) -> 311-470LRTR-ND; Supplier Part Num 3 (none) -> C114877
Connections:
- net +3.3V: no longer R1.1, R2.1
- net GND: now also LED2.1 (K); no longer LED2.C
- net LED-ACT: now also U1.12 (GPIO2)
- net LED-LINK: now also LED1.1 (K), U1.9 (GPIO0); no longer LED1.C
- net LED-SELFCHECK: now also U1.10 (GPIO1)
- net PE-RD+: now also U1.15 (PERX_P)
- net PE-RD-: now also U1.16 (PERX_N)
- net PE-TD+: now also U1.18 (PETX_P)
- net PE-TD-: now also U1.19 (PETX_N)
- net PL_L: now also T1.5 (PL_L)
- net PL_N: now also T1.8 (PL_N)
- net RX+: now also T1.1 (RX+), U1.5 (RX+)
- net RX-: now also T1.4 (RX-), U1.6 (RX-)
- net TX+: now also C2.2, T1.2 (TX+), U1.2 (TX+); no longer C2.1
- net TX-: now also C2.1, T1.3 (TX-), U1.3 (TX-); no longer C2.2
- net VDD2P0: now also U1.14 (VDD2P0)
- net at R2.2: now also LED2.2 (A); no longer LED2.A
- net at R1.2: now also LED1.2 (A); no longer LED1.A
- new net 3V3: R1.1, R2.1, U1.20 (3.3VD)
- new net GNDREF: U1.1 (GND), U1.11 (GND), U1.17 (GND), U1.4 (GND), U1.7 (GND)
- new net nRST: U1.13 (GPIO3)
- no-connect marks 0 -> 1
Other:
- moved on the sheet: C1, C2, C3, C4, C5, C6, D1, IC1, JP2, R3, R4, R5
